File: KiCad/Isolation.sch (KiCad schematic (older format))
At the start: 5 parts, among them U19 Si8642BA-B-IU

Commit message: Many small fixes
Changed lines of the file:
@@
 AR Path="/5C982601/5C9D2CA8/5D2AE2CA" Ref="U19"  Part="1"
 AR Path="/5CA35A27/5CA7F8E1/5D2AE2CA" Ref="U13"  Part="1"
-F 0 "U19" H 5250 3967 50  0000 C CNN
+F 0 "U13" H 5250 3967 50  0000 C CNN
 F 1 "Si8642BA-B-IU" H 5250 3876 50  0000 C CNN
 F 2 "Package_SO:QSOP-16_3.9x4.9mm_P0.635mm" H 5250 3875 50  0001 C CIN
@@
 AR Path="/5C982601/5C9D2CA8/5D2AE2D1" Ref="RN18"  Part="1"
 AR Path="/5CA35A27/5CA7F8E1/5D2AE2D1" Ref="RN11"  Part="1"
-F 0 "RN18" V 4050 3400 50  0000 C CNN
+F 0 "RN11" V 4050 3400 50  0000 C CNN
 F 1 "R_Pack02" V 4050 3400 50  0001 C CNN
 F 2 "Resistor_SMD:R_Array_Convex_2x0402" V 4425 3400 50  0001 C CNN
@@
 AR Path="/5C982601/5C9D2CA8/5D7B4823" Ref="C51"  Part="1"
 AR Path="/5CA35A27/5CA7F8E1/5D7B4823" Ref="C44"  Part="1"
-F 0 "C51" H 3615 3396 50  0000 L CNN
+F 0 "C44" H 3615 3396 50  0000 L CNN
 F 1 "1uF" H 3615 3305 50  0000 L CNN
 F 2 "Capacitor_SMD:C_0603_1608Metric_Pad1.05x0.95mm_HandSolder" H 3538 3200 50  0001 C CNN
@@
 AR Path="/5C982601/5C9D2CA8/5D7B4959" Ref="C52"  Part="1"
 AR Path="/5CA35A27/5CA7F8E1/5D7B4959" Ref="C45"  Part="1"
-F 0 "C52" H 6615 3396 50  0000 L CNN
+F 0 "C45" H 6615 3396 50  0000 L CNN
 F 1 "1uF" H 6615 3305 50  0000 L CNN
 F 2 "Capacitor_SMD:C_0603_1608Metric_Pad1.05x0.95mm_HandSolder" H 6538 3200 50  0001 C CNN
@@
 AR Path="/5C982601/5C9D2CA8/5C319048" Ref="RN19"  Part="1"
 AR Path="/5CA35A27/5CA7F8E1/5C319048" Ref="RN12"  Part="1"
-F 0 "RN19" V 4450 4000 50  0000 C CNN
+F 0 "RN12" V 4450 4000 50  0000 C CNN
 F 1 "R_Pack02" V 4450 4000 50  0001 C CNN
 F 2 "Resistor_SMD:R_Array_Convex_2x0402" V 4825 4000 50  0001 C CNN
