File: KiCad/Tile0.sch (KiCad schematic (older format))
At the start: 18 parts, among them J15 Conn_02x08_Odd_Even, SW2 BOOT, SW3 GP, U9 XUF216-512-FB236

Commit message: Update
Updated to KiCad 5.1.6 and changed the power sheet etc.
Parts:
- U9: symbol xmos:XUF216-512-FB236 -> XMOS_XUF216_FB236-rescue:XUF216-512-FB236-xmos-XMOS_XUF216_FB236-rescue
Changed lines of the file:
@@
 EESchema Schematic File Version 4
-LIBS:XMOS_XUF216_FB236-cache
-EELAYER 26 0
+EELAYER 30 0
 EELAYER END
 $Descr A4 11693 8268
@@
 Sheet 11 16
 Title "XMOS Tile0"
-Date "2019-01-08"
+Date "2020-06-05"
 Rev "BETA"
 Comp "openPnP"
@@
 $EndDescr
 $Comp
-L xmos:XUF216-512-FB236 U?
+L XMOS_XUF216_FB236-rescue:XUF216-512-FB236-xmos-XMOS_XUF216_FB236-rescue U?
 U 3 1 5C99BC42
 P 10300 4050
@@
 2 x 3 phase + watchdog =7 pins
 $Comp
-L xmos:XUF216-512-FB236 U?
+L XMOS_XUF216_FB236-rescue:XUF216-512-FB236-xmos-XMOS_XUF216_FB236-rescue U?
 U 2 1 5C9D2BFC
 P 3900 5300
