File: KiCad/Tile1.sch (KiCad schematic (older format))
At the start: 7 parts, among them J11 Conn_02x12_Odd_Even, J6 Conn_02x08_Odd_Even, U9 XUF216-512-FB236

Commit message: Update
Updated to KiCad 5.1.6 and changed the power sheet etc.
Parts:
- U9: symbol xmos:XUF216-512-FB236 -> XMOS_XUF216_FB236-rescue:XUF216-512-FB236-xmos-XMOS_XUF216_FB236-rescue
Changed lines of the file:
@@
 EESchema Schematic File Version 4
-LIBS:XMOS_XUF216_FB236-cache
-EELAYER 26 0
+EELAYER 30 0
 EELAYER END
 $Descr A4 11693 8268
@@
 Sheet 7 16
 Title "XMOS Tile1"
-Date "2019-01-08"
+Date "2020-06-05"
 Rev "BETA"
 Comp "openPnP"
@@
 ETH.PHY_RSTn
 $Comp
-L xmos:XUF216-512-FB236 U?
+L XMOS_XUF216_FB236-rescue:XUF216-512-FB236-xmos-XMOS_XUF216_FB236-rescue U?
 U 5 1 5CA63C77
 P 9850 4300
@@
 $EndComp
 $Comp
-L xmos:XUF216-512-FB236 U?
+L XMOS_XUF216_FB236-rescue:XUF216-512-FB236-xmos-XMOS_XUF216_FB236-rescue U?
 U 4 1 5CA7F845
 P 3250 4350
