File: KiCad/power.sch (KiCad schematic (older format))
At the start: 54 parts, among them J2 Barrel_Jack_MountingPin, J3 Conn_01x04, M1 RFM-0505S, SW1 RESET, U2 IC-RES-TPS3808, U3 IC-REG-ST1S06, U4 IC-REG-ST1S06, U5 IC-LOGIC-BUF-NC7WZ04P6X, U6 LM2574HVM-5, U7 MIC5504-3.3YM5

Commit message: Added impedance calc, and rerouted USB
Parts:
- U5: footprint MyKiCadLibs-Footprints:IC-SC70-6 -> Package_TO_SOT_SMD:SOT-363_SC-70-6_Handsoldering
Changed lines of the file:
@@
 F 0 "U5" H 4675 6537 60  0000 C CNN
 F 1 "IC-LOGIC-BUF-NC7WZ04P6X" H 4675 6431 60  0000 C CNN
-F 2 "MyKiCadLibs-Footprints:IC-SC70-6" H 5650 6150 60  0001 C CNN
+F 2 "Package_TO_SOT_SMD:SOT-363_SC-70-6_Handsoldering" H 5650 6150 60  0001 C CNN
 F 3 "" H 4750 6250 60  0000 C CNN
 F 4 "NC7WZ04 TinyLogic UHS Dual Inverter" H 5700 6250 60  0001 C CNN "Decription"
@@
 F 0 "U5" H 6278 6753 60  0000 L CNN
 F 1 "IC-LOGIC-BUF-NC7WZ04P6X" H 6200 7200 60  0000 L CNN
-F 2 "MyKiCadLibs-Footprints:IC-SC70-6" H 7100 6600 60  0001 C CNN
+F 2 "Package_TO_SOT_SMD:SOT-363_SC-70-6_Handsoldering" H 7100 6600 60  0001 C CNN
 F 3 "" H 6200 6700 60  0000 C CNN
 F 4 "NC7WZ04 TinyLogic UHS Dual Inverter" H 7150 6700 60  0001 C CNN "Decription"
@@
 F 0 "U5" V 825 6471 60  0000 R CNN
 F 1 "IC-LOGIC-BUF-NC7WZ04P6X" V 771 6471 60  0001 R CNN
-F 2 "MyKiCadLibs-Footprints:IC-SC70-6" H 1800 6500 60  0001 C CNN
+F 2 "Package_TO_SOT_SMD:SOT-363_SC-70-6_Handsoldering" H 1800 6500 60  0001 C CNN
 F 3 "" H 900 6600 60  0000 C CNN
 F 4 "NC7WZ04 TinyLogic UHS Dual Inverter" H 1850 6600 60  0001 C CNN "Decription"

Commit message: Many small fixes
Connections:
- net Vin: now reaches C10.1, F1.1, TP6.1, U6.10 (VIN)
- net FB5V: now reaches C13.1, FB2.2, L3.1, U6.3 (FB)
- net F: now reaches D3.1 (K), F1.2
Changed lines of the file:
@@
 $EndComp
 NoConn ~ 800  6300
+Text Label 8075 2100 0    50   ~ 0
+F
+Text Label 9725 2100 0    50   ~ 0
+FB5V
+Text Label 8500 2100 0    50   ~ 0
+Vin
 $EndSCHEMATC
