File: KiCad/power.sch (KiCad schematic (older format))
At the start: 54 parts, among them J2 Barrel_Jack_MountingPin, J3 Conn_01x04, M1 RFM-0505S, SW1 RESET, U2 IC-RES-TPS3808, U3 IC-REG-ST1S06, U4 IC-REG-ST1S06, U5 IC-LOGIC-BUF-NC7WZ04P6X, U6 LM2574HVM-5, U7 MIC5504-3.3YM5

Commit message: Update
Updated to KiCad 5.1.6 and changed the power sheet etc.
Parts:
- removed C9: C, Capacitor_SMD:C_0603_1608Metric_Pad1.05x0.95mm_HandSolder, symbol Device:C
- removed U5: IC-LOGIC-BUF-NC7WZ04P6X, Package_TO_SOT_SMD:SOT-363_SC-70-6_Handsoldering, symbol MyKiCadLibs-Lib:IC-LOGIC-BUF-NC7WZ04P6X
- added R59: 130k, Resistor_SMD:R_0603_1608Metric_Pad1.05x0.95mm_HandSolder, symbol Device:R
- C10: Voltage (none) -> 100V
- C5: value 10nF -> 1nF
- D1: value GREEN -> RED
- M1: symbol xmos_project:RFM-0505S -> XMOS_XUF216_FB236-rescue:RFM-0505S-xmos_project-XMOS_XUF216_FB236-rescue
- R5: value 10k -> 27k
- R6: value 7k5 -> 10k
- U2: value IC-RES-TPS3808 -> TPS3808G01; symbol MyKiCadLibs-Lib:IC-RES-TPS3808 -> XMOS_XUF216_FB236-rescue:IC-RES-TPS3808-MyKiCadLibs-Lib-XMOS_XUF216_FB236-rescue
- U3, U4: symbol MyKiCadLibs-Lib:IC-REG-ST1S06 -> XMOS_XUF216_FB236-rescue:IC-REG-ST1S06-MyKiCadLibs-Lib-XMOS_XUF216_FB236-rescue
Connections:
- net LVDS_EN is gone; now on an unnamed net: D1.2 (A)
- net +3V3: now also R7.1, R59.2; no longer U4.6 (EN)
- net +5V: now also U4.6 (EN)
- net GND: no longer R7.1
- net SENSE: now also R59.1
- net ~RST: now also D1.1 (K)
- net at R7.2: no longer D1.1 (K)
- no-connect marks 2 -> 1
Other:
- note added: "200nA\n"
- moved on the sheet: D1, R7
