File: KiCad/LVDS.sch (KiCad schematic (older format))
At the start: 7 parts, among them J1 RJ45_Shielded, U1 DS90LV049TMT

Commit message: Update
Updated to KiCad 5.1.6 and changed the power sheet etc.
Parts:
- U1: symbol xmos_project:DS90LV049TMT -> XMOS_XUF216_FB236-rescue:DS90LV049TMT-xmos_project-XMOS_XUF216_FB236-rescue
Changed lines of the file:
@@
 EESchema Schematic File Version 4
-LIBS:XMOS_XUF216_FB236-cache
-EELAYER 26 0
+EELAYER 30 0
 EELAYER END
 $Descr A4 11693 8268
@@
 Sheet 16 16
 Title "LVDS <-> Xlinks"
-Date "2019-01-08"
+Date "2020-06-05"
 Rev "BETA"
 Comp "openPnP"
@@
 AR Path="/5CAE894D/5C318F8C" Ref="J14"  Part="1"
 AR Path="/5CC36DF5/5C318F8C" Ref="J19"  Part="1"
-F 0 "J4" H 4246 3016 50  0000 R CNN
+F 0 "J19" H 4246 3016 50  0000 R CNN
 F 1 "RJ45_Shielded" H 4246 2925 50  0000 R CNN
 F 2 "Connector_RJ:RJ45_Amphenol_RJHSE5380" V 4575 3000 50  0001 C CNN
@@
 IN0
 $Comp
-L xmos_project:DS90LV049TMT U?
+L XMOS_XUF216_FB236-rescue:DS90LV049TMT-xmos_project-XMOS_XUF216_FB236-rescue U?
 U 1 1 5C1F0997
 P 2625 3075
@@
 AR Path="/5CAE894D/5C1F0997" Ref="U15"  Part="1"
 AR Path="/5CC36DF5/5C1F0997" Ref="U20"  Part="1"
-F 0 "U8" H 2525 3325 50  0000 L CNN
+AR Path="/5C1F0997" Ref="U20"  Part="1"
+F 0 "U20" H 2525 3325 50  0000 L CNN
 F 1 "DS90LV049TMT" H 2925 2125 50  0000 L CNN
 F 2 "Package_SO:TSSOP-16_4.4x5mm_P0.65mm" H 2625 3075 50  0001 C CNN
@@
 AR Path="/5CAE894D/5C318FC1" Ref="C47"  Part="1"
 AR Path="/5CC36DF5/5C318FC1" Ref="C53"  Part="1"
-F 0 "C15" H 1840 4521 50  0000 L CNN
+F 0 "C53" H 1840 4521 50  0000 L CNN
 F 1 "100nF" H 1840 4430 50  0000 L CNN
 F 2 "Capacitor_SMD:C_0603_1608Metric_Pad1.05x0.95mm_HandSolder" H 1763 4325 50  0001 C CNN
@@
 AR Path="/5CAE894D/5E2282E6" Ref="R37"  Part="1"
 AR Path="/5CC36DF5/5E2282E6" Ref="R56"  Part="1"
-F 0 "R17" H 4145 4021 50  0000 L CNN
+F 0 "R56" H 4145 4021 50  0000 L CNN
 F 1 "100R" H 4145 3930 50  0000 L CNN
 F 2 "Resistor_SMD:R_0402_1005Metric" V 4005 3975 50  0001 C CNN
@@
 AR Path="/5CAE894D/5E22A193" Ref="R38"  Part="1"
 AR Path="/5CC36DF5/5E22A193" Ref="R57"  Part="1"
-F 0 "R18" H 4595 3771 50  0000 L CNN
+F 0 "R57" H 4595 3771 50  0000 L CNN
 F 1 "100R" H 4595 3680 50  0000 L CNN
 F 2 "Resistor_SMD:R_0402_1005Metric" V 4455 3725 50  0001 C CNN
@@
 AR Path="/5CAE894D/5C319046" Ref="R36"  Part="1"
 AR Path="/5CC36DF5/5C319046" Ref="R55"  Part="1"
-F 0 "R16" H 2295 2721 50  0000 L CNN
+F 0 "R55" H 2295 2721 50  0000 L CNN
 F 1 "47k" H 2295 2630 50  0000 L CNN
 F 2 "Resistor_SMD:R_0402_1005Metric" V 2155 2675 50  0001 C CNN
@@
 AR Path="/5CAE894D/5E5F7C9F" Ref="R35"  Part="1"
 AR Path="/5CC36DF5/5E5F7C9F" Ref="R54"  Part="1"
-F 0 "R15" H 1945 2721 50  0000 L CNN
+F 0 "R54" H 1945 2721 50  0000 L CNN
 F 1 "47k" H 1945 2630 50  0000 L CNN
 F 2 "Resistor_SMD:R_0402_1005Metric" V 1805 2675 50  0001 C CNN
