File: KiCad/XMOS_USB.sch (KiCad schematic (older format))
At the start: 31 parts, among them J5 USB_B_Mini, U10 TPD2E2U06, U9 XUF216-512-FB236, X1 ASV-24MHz

Commit message: Update
Updated to KiCad 5.1.6 and changed the power sheet etc.
Parts:
- U9: symbol xmos:XUF216-512-FB236 -> XMOS_XUF216_FB236-rescue:XUF216-512-FB236-xmos-XMOS_XUF216_FB236-rescue
Changed lines of the file:
@@
 EESchema Schematic File Version 4
-LIBS:XMOS_XUF216_FB236-cache
-EELAYER 26 0
+EELAYER 30 0
 EELAYER END
 $Descr A4 11693 8268
@@
 Sheet 5 16
 Title "XTAG & XMOS USB"
-Date "2019-01-08"
+Date "2020-06-05"
 Rev "BETA"
 Comp "openPnP"
@@
 $EndComp
 $Comp
-L xmos:XUF216-512-FB236 U?
+L XMOS_XUF216_FB236-rescue:XUF216-512-FB236-xmos-XMOS_XUF216_FB236-rescue U?
 U 1 1 5C4CC3CE
 P 6250 4700
