File: KiCad/XTAG.sch (KiCad schematic (older format))
At the start: 28 parts, among them J10 Conn_02x10_FEMALE_toNext, J7 Mini-DIN-8, J8 Conn_02x10_MALE_FROM_XTAG, J9 Mini-DIN-8, U11 NC7WZ17, U12 NC7SZ157

Commit message: Update
Updated to KiCad 5.1.6 and changed the power sheet etc.
Parts:
- U11: symbol xmos_project:NC7WZ17 -> XMOS_XUF216_FB236-rescue:NC7WZ17-xmos_project-XMOS_XUF216_FB236-rescue
- U12: symbol xmos_project:NC7SZ157 -> XMOS_XUF216_FB236-rescue:NC7SZ157-xmos_project-XMOS_XUF216_FB236-rescue
Changed lines of the file:
@@
 EESchema Schematic File Version 4
-LIBS:XMOS_XUF216_FB236-cache
-EELAYER 26 0
+EELAYER 30 0
 EELAYER END
 $Descr A4 11693 8268
@@
 Sheet 6 16
 Title "XTAG / xSYS"
-Date "2019-01-08"
+Date "2020-06-05"
 Rev "BETA"
 Comp "openPnP"
@@
 XTAG.MSEL
 $Comp
-L xmos_project:NC7SZ157 U?
+L XMOS_XUF216_FB236-rescue:NC7SZ157-xmos_project-XMOS_XUF216_FB236-rescue U?
 U 1 1 5C7707A3
 P 5250 3700
@@
 A connected header or mini DIN will ground this net
 $Comp
-L xmos_project:NC7WZ17 U?
+L XMOS_XUF216_FB236-rescue:NC7WZ17-xmos_project-XMOS_XUF216_FB236-rescue U?
 U 1 1 5C7707CC
 P 3450 2350
